Commit message: Add static transforms from FSD to FLU

File: hardware/autonomy_pi/ros/autonomy_description/description/ros2_control/ros2_control.xacro (robot description, xacro)
@@ -1,5 +1,8 @@
-<?xml version="1.0"?>
+<?xml version="1.0" ?>
 <robot xmlns:xacro="http://www.ros.org/wiki/xacro">
-  <xacro:macro name="bluerov2_system" params="prefix max_set_param_attempts:=^3">
+  <xacro:macro
+        name="bluerov2_system"
+        params="prefix max_set_param_attempts:=^3"
+    >
     <!-- BlueROV2 thruster system -->
     <ros2_control name="thruster_control_system" type="system">

File: hardware/autonomy_pi/ros/autonomy_description/description/urdf/bluerov2.urdf.xacro (robot description, xacro)
@@ -1,3 +1,3 @@
-<?xml version="1.0"?>
+<?xml version="1.0" ?>
 <robot xmlns:xacro="http://ros.org/wiki/xacro">
   <xacro:macro name="bluerov2_urdf" params="prefix">
@@ -7,12 +7,5 @@
         <origin rpy="0 0 0" xyz="0.0 0.0 0.0" />
         <mass value="15.0" />
-        <inertia
-          ixx="0.26"
-          ixy="0"
-          ixz="0"
-          iyy="0.23"
-          iyz="0"
-          izz="0.37"
-        />
+        <inertia ixx="0.26" ixy="0" ixz="0" iyy="0.23" iyz="0" izz="0.37" />
       </inertial>
       <collision name="base_link_collision">
@@ -36,9 +29,4 @@
       <child link="${prefix}dvl_link" />
     </joint>
-    <joint name="${prefix}locator_joint" type="fixed">
-      <origin rpy="3.141593 0 0" xyz="0.023365 0.174609 0.188394" />
-      <parent link="${prefix}base_link" />
-      <child link="${prefix}locator_link" />
-    </joint>
     <joint name="${prefix}bno08x_joint" type="fixed">
       <origin rpy="0 0 -1.57079633" xyz="0.029369 0.02235 -0.115472" />
@@ -52,27 +40,69 @@
     </joint>
     <!-- Import T200 macro -->
-    <xacro:include filename="$(find autonomy_description)/description/urdf/t200.urdf.xacro" />
-    <xacro:t200_urdf parent="${prefix}base_link" prefix="${prefix}" ccw="true" id="1">
+    <xacro:include
+            filename="$(find autonomy_description)/description/urdf/t200.urdf.xacro"
+        />
+    <xacro:t200_urdf
+            parent="${prefix}base_link"
+            prefix="${prefix}"
+            ccw="true"
+            id="1"
+        >
       <origin rpy="-1.571 1.571 -1.047" xyz="0.09 -0.104 0.0" />
     </xacro:t200_urdf>
-    <xacro:t200_urdf parent="${prefix}base_link" prefix="${prefix}" ccw="true" id="2">
+    <xacro:t200_urdf
+            parent="${prefix}base_link"
+            prefix="${prefix}"
+            ccw="true"
+            id="2"
+        >
       <origin rpy="-1.571 1.571 -2.094" xyz="0.09 0.104 0.0" />
     </xacro:t200_urdf>
-    <xacro:t200_urdf parent="${prefix}base_link" prefix="${prefix}" ccw="false" id="3">
+    <xacro:t200_urdf
+            parent="${prefix}base_link"
+            prefix="${prefix}"
+            ccw="false"
+            id="3"
+        >
       <origin rpy="-1.571 1.571 1.047" xyz="-0.09 -0.104 0.0" />
     </xacro:t200_urdf>
-    <xacro:t200_urdf parent="${prefix}base_link" prefix="${prefix}" ccw="false" id="4">
+    <xacro:t200_urdf
+            parent="${prefix}base_link"
+            prefix="${prefix}"
+            ccw="false"
+            id="4"
+        >
       <origin rpy="-1.571 1.571 2.094" xyz="-0.09 0.104 0.0" />
     </xacro:t200_urdf>
-    <xacro:t200_urdf parent="${prefix}base_link" prefix="${prefix}" ccw="true" id="5">
+    <xacro:t200_urdf
+            parent="${prefix}base_link"
+            prefix="${prefix}"
+            ccw="true"
+            id="5"
+        >
       <origin rpy="0 0 0" xyz="0.12 -0.218 0.11" />
     </xacro:t200_urdf>
-    <xacro:t200_urdf parent="${prefix}base_link" prefix="${prefix}" ccw="false" id="6">
+    <xacro:t200_urdf
+            parent="${prefix}base_link"
+            prefix="${prefix}"
+            ccw="false"
+            id="6"
+        >
       <origin rpy="0 0 0" xyz="0.12 0.218 0.11" />
     </xacro:t200_urdf>
-    <xacro:t200_urdf parent="${prefix}base_link" prefix="${prefix}" ccw="false" id="7">
+    <xacro:t200_urdf
+            parent="${prefix}base_link"
+            prefix="${prefix}"
+            ccw="false"
+            id="7"
+        >
       <origin rpy="0 0 0" xyz="-0.12 -0.218 0.11" />
     </xacro:t200_urdf>
-    <xacro:t200_urdf parent="${prefix}base_link" prefix="${prefix}" ccw="true" id="8">
+    <xacro:t200_urdf
+            parent="${prefix}base_link"
+            prefix="${prefix}"
+            ccw="true"
+            id="8"
+        >
       <origin rpy="0 0 0" xyz="-0.12 0.218 0.11" />
     </xacro:t200_urdf>
