Commit message: save

File: hardware/autonomy_pi/ros/autonomy_description/description/urdf/bluerov2.urdf.xacro (robot description, xacro)
@@ -17,5 +17,4 @@
     </link>
     <link name="${prefix}dvl_link" />
-    <link name="${prefix}locator_link" />
     <link name="${prefix}bno08x" />
     <link name="${prefix}bar30" />
