Commit message: formatting

File: modules/autonomy_pi/ros/autonomy_description/description/config.xacro (robot description, xacro)
@@ -1,3 +1,3 @@
-<?xml version="1.0"?>
+<?xml version="1.0" ?>
 <robot name="bluerov2" xmlns:xacro="http://ros.org/wiki/xacro">
   <xacro:include filename="$(find autonomy_description)/description/urdf/bluerov2.urdf.xacro" />

File: modules/autonomy_pi/ros/autonomy_description/description/ros2_control/ros2_control.xacro (robot description, xacro)
@@ -1,8 +1,5 @@
 <?xml version="1.0" ?>
 <robot xmlns:xacro="http://www.ros.org/wiki/xacro">
-  <xacro:macro
-        name="bluerov2_system"
-        params="prefix max_set_param_attempts:=^3"
-    >
+  <xacro:macro name="bluerov2_system" params="prefix max_set_param_attempts:=^3">
     <!-- BlueROV2 thruster system -->
     <ros2_control name="thruster_control_system" type="system">

File: modules/autonomy_pi/ros/autonomy_description/description/urdf/bluerov2.urdf.xacro (robot description, xacro)
@@ -39,69 +39,27 @@
     </joint>
     <!-- Import T200 macro -->
-    <xacro:include
-            filename="$(find autonomy_description)/description/urdf/t200.urdf.xacro"
-        />
-    <xacro:t200_urdf
-            parent="${prefix}base_link"
-            prefix="${prefix}"
-            ccw="true"
-            id="1"
-        >
+    <xacro:include filename="$(find autonomy_description)/description/urdf/t200.urdf.xacro" />
+    <xacro:t200_urdf parent="${prefix}base_link" prefix="${prefix}" ccw="true" id="1">
       <origin rpy="-1.571 1.571 -1.047" xyz="0.09 -0.104 0.0" />
     </xacro:t200_urdf>
-    <xacro:t200_urdf
-            parent="${prefix}base_link"
-            prefix="${prefix}"
-            ccw="true"
-            id="2"
-        >
+    <xacro:t200_urdf parent="${prefix}base_link" prefix="${prefix}" ccw="true" id="2">
       <origin rpy="-1.571 1.571 -2.094" xyz="0.09 0.104 0.0" />
     </xacro:t200_urdf>
-    <xacro:t200_urdf
-            parent="${prefix}base_link"
-            prefix="${prefix}"
-            ccw="false"
-            id="3"
-        >
+    <xacro:t200_urdf parent="${prefix}base_link" prefix="${prefix}" ccw="false" id="3">
       <origin rpy="-1.571 1.571 1.047" xyz="-0.09 -0.104 0.0" />
     </xacro:t200_urdf>
-    <xacro:t200_urdf
-            parent="${prefix}base_link"
-            prefix="${prefix}"
-            ccw="false"
-            id="4"
-        >
+    <xacro:t200_urdf parent="${prefix}base_link" prefix="${prefix}" ccw="false" id="4">
       <origin rpy="-1.571 1.571 2.094" xyz="-0.09 0.104 0.0" />
     </xacro:t200_urdf>
-    <xacro:t200_urdf
-            parent="${prefix}base_link"
-            prefix="${prefix}"
-            ccw="true"
-            id="5"
-        >
+    <xacro:t200_urdf parent="${prefix}base_link" prefix="${prefix}" ccw="true" id="5">
       <origin rpy="0 0 0" xyz="0.12 -0.218 0.11" />
     </xacro:t200_urdf>
-    <xacro:t200_urdf
-            parent="${prefix}base_link"
-            prefix="${prefix}"
-            ccw="false"
-            id="6"
-        >
+    <xacro:t200_urdf parent="${prefix}base_link" prefix="${prefix}" ccw="false" id="6">
       <origin rpy="0 0 0" xyz="0.12 0.218 0.11" />
     </xacro:t200_urdf>
-    <xacro:t200_urdf
-            parent="${prefix}base_link"
-            prefix="${prefix}"
-            ccw="false"
-            id="7"
-        >
+    <xacro:t200_urdf parent="${prefix}base_link" prefix="${prefix}" ccw="false" id="7">
       <origin rpy="0 0 0" xyz="-0.12 -0.218 0.11" />
     </xacro:t200_urdf>
-    <xacro:t200_urdf
-            parent="${prefix}base_link"
-            prefix="${prefix}"
-            ccw="true"
-            id="8"
-        >
+    <xacro:t200_urdf parent="${prefix}base_link" prefix="${prefix}" ccw="true" id="8">
       <origin rpy="0 0 0" xyz="-0.12 0.218 0.11" />
     </xacro:t200_urdf>

File: modules/autonomy_pi/ros/autonomy_description/description/urdf/t200.urdf.xacro (robot description, xacro)
@@ -1,3 +1,3 @@
-<?xml version="1.0"?>
+<?xml version="1.0" ?>
 <robot xmlns:xacro="http://ros.org/wiki/xacro">
   <xacro:macro name="t200_urdf" params="prefix id parent *origin ccw:=^false">
@@ -5,12 +5,5 @@
       <inertial>
         <mass value="0.002" />
-        <inertia
-          ixx="0.001"
-          ixy="0"
-          ixz="0"
-          iyy="0.001"
-          iyz="0"
-          izz="0.001"
-        />
+        <inertia ixx="0.001" ixy="0" ixz="0" iyy="0.001" iyz="0" izz="0.001" />
       </inertial>
     </link>
