Commit message: TEST POINT

File: modules/autonomy_pi/ros/autonomy_description/description/urdf/bluerov2.urdf.xacro (robot description, xacro)
@@ -29,5 +29,5 @@
     </joint>
     <joint name="${prefix}bno08x_joint" type="fixed">
-      <origin rpy="0 0 -1.57079633" xyz="0.029369 0.02235 -0.115472" />
+      <origin rpy="0 0 1.57079633" xyz="0.029369 0.02235 -0.115472" />
       <parent link="${prefix}base_link" />
       <child link="${prefix}bno08x" />

Commit message: Fix networking and add services to boot system on startup (#18)
* Rewrite networking for BlueROV Pi based on latest image.

* fix permissions

* Fix the platform type in the compose script

* cleanup

* bump changelogs

* fix gpiochip and readme

* fix launch

* split launch files and added notes

* Address bug in TAM

* starting jetson install scripts

* Add jetson module

* TEST POINT

* Add deployment services to autonomy pi

* Cleanup

* Improve IMU calibration UI

* Fixes for DVL and reset-ekf

* dvl fixes and prep for data collection

* Tuning EKF and controllers

* formatting

* Remove passwords from networking

* Address initial PR comments

* remove pycache

* removed stale dir

* Fix readme

* Use local install instead of docker

* bump release version

File: modules/autonomy_pi/ros/autonomy_description/description/urdf/bluerov2.urdf.xacro (robot description, xacro)
@@ -29,5 +29,5 @@
     </joint>
     <joint name="${prefix}bno08x_joint" type="fixed">
-      <origin rpy="0 0 -1.57079633" xyz="0.029369 0.02235 -0.115472" />
+      <origin rpy="0 0 1.57079633" xyz="0.029369 0.02235 -0.115472" />
       <parent link="${prefix}base_link" />
       <child link="${prefix}bno08x" />
@@ -39,69 +39,27 @@
     </joint>
     <!-- Import T200 macro -->
-    <xacro:include
-            filename="$(find autonomy_description)/description/urdf/t200.urdf.xacro"
-        />
-    <xacro:t200_urdf
-            parent="${prefix}base_link"
-            prefix="${prefix}"
-            ccw="true"
-            id="1"
-        >
+    <xacro:include filename="$(find autonomy_description)/description/urdf/t200.urdf.xacro" />
+    <xacro:t200_urdf parent="${prefix}base_link" prefix="${prefix}" ccw="true" id="1">
       <origin rpy="-1.571 1.571 -1.047" xyz="0.09 -0.104 0.0" />
     </xacro:t200_urdf>
-    <xacro:t200_urdf
-            parent="${prefix}base_link"
-            prefix="${prefix}"
-            ccw="true"
-            id="2"
-        >
+    <xacro:t200_urdf parent="${prefix}base_link" prefix="${prefix}" ccw="true" id="2">
       <origin rpy="-1.571 1.571 -2.094" xyz="0.09 0.104 0.0" />
     </xacro:t200_urdf>
-    <xacro:t200_urdf
-            parent="${prefix}base_link"
-            prefix="${prefix}"
-            ccw="false"
-            id="3"
-        >
+    <xacro:t200_urdf parent="${prefix}base_link" prefix="${prefix}" ccw="false" id="3">
       <origin rpy="-1.571 1.571 1.047" xyz="-0.09 -0.104 0.0" />
     </xacro:t200_urdf>
-    <xacro:t200_urdf
-            parent="${prefix}base_link"
-            prefix="${prefix}"
-            ccw="false"
-            id="4"
-        >
+    <xacro:t200_urdf parent="${prefix}base_link" prefix="${prefix}" ccw="false" id="4">
       <origin rpy="-1.571 1.571 2.094" xyz="-0.09 0.104 0.0" />
     </xacro:t200_urdf>
-    <xacro:t200_urdf
-            parent="${prefix}base_link"
-            prefix="${prefix}"
-            ccw="true"
-            id="5"
-        >
+    <xacro:t200_urdf parent="${prefix}base_link" prefix="${prefix}" ccw="true" id="5">
       <origin rpy="0 0 0" xyz="0.12 -0.218 0.11" />
     </xacro:t200_urdf>
-    <xacro:t200_urdf
-            parent="${prefix}base_link"
-            prefix="${prefix}"
-            ccw="false"
-            id="6"
-        >
+    <xacro:t200_urdf parent="${prefix}base_link" prefix="${prefix}" ccw="false" id="6">
       <origin rpy="0 0 0" xyz="0.12 0.218 0.11" />
     </xacro:t200_urdf>
-    <xacro:t200_urdf
-            parent="${prefix}base_link"
-            prefix="${prefix}"
-            ccw="false"
-            id="7"
-        >
+    <xacro:t200_urdf parent="${prefix}base_link" prefix="${prefix}" ccw="false" id="7">
       <origin rpy="0 0 0" xyz="-0.12 -0.218 0.11" />
     </xacro:t200_urdf>
-    <xacro:t200_urdf
-            parent="${prefix}base_link"
-            prefix="${prefix}"
-            ccw="true"
-            id="8"
-        >
+    <xacro:t200_urdf parent="${prefix}base_link" prefix="${prefix}" ccw="true" id="8">
       <origin rpy="0 0 0" xyz="-0.12 0.218 0.11" />
     </xacro:t200_urdf>
